File: pcb/sterna.kicad_pcb (KiCad board)
At the start: 2 copper layers, 232.3 x 107.8 mm, 75 parts

Commit message: Add files via upload
Parts:
- B1: footprint Panasonic_EVQPUL_EVQPUC -> Button_Switch_SMD:Panasonic_EVQPUL_EVQPUC
- PAD1, PAD2, PAD3, PAD4: footprint MountingHole_2.2mm_M2_Pad -> MountingHole:MountingHole_2.2mm_M2_Pad
- PAD10, PAD5, PAD6, PAD7, PAD8, PAD9: footprint MountingHole_2.2mm_M2 -> MountingHole:MountingHole_2.2mm_M2
- S1, S10, S11, S12, S13, S14, S15, S16, S17, S18, S19, S2, S20, S21, S22, S23, S24, S25, S26, S27, S28, S29, S3, S30, S4, S5, S6, S7, S8, S9: footprint PG1350 -> Library-keyswitches:Kailh_socket_PG1350
- moved S16 8.41 mm to (262.2, 130.1)
- moved S29 8.41 mm to (220.6, 167.8)
- moved PAD6 8.41 mm to (212.6, 173.1)
- moved D28 8.41 mm to (147.9, 182.1)
- moved S26 8.41 mm to (202.1, 127.3)
- moved S22 8.41 mm to (228.2, 142.8)
- moved PAD7 8.41 mm to (112.3, 101.6)
- moved D26 8.41 mm to (203.9, 131.6)
- moved PAD3 8.41 mm to (151.5, 162.9)
- moved PAD5 8.41 mm to (142.8, 173.1)
- moved D17 8.41 mm to (258.8, 118.3)
- moved S2 8.41 mm to (75.3, 118.3)
- moved S5 8.41 mm to (102.6, 97.4)
- moved D3 8.41 mm to (91.9, 134.6)
- moved D11 8.41 mm to (138.6, 115.9)
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